File: kbpcb/pcb/Citrouille90/citrouille90.kicad_pcb (KiCad board)
At the start: 2 copper layers, 386.7 x 125.7 mm, 200 parts, among them J1 3 pin connector, J3 USB mini b connector, U1 AVR64DU32-I/PT, U2 USBLC6-2SC6

Commit message: PCB work
Parts:
- added C3: 4.7n, capacitors:C_0805_2012Metric_Pad1.18x1.45mm_HandSolder, B.Cu at (-9.36, -61.3)
- added H1: Mechanical_MountingHole, MountingHole:MountingHole_2.7mm_M2.5_ISO7380_Pad, F.Cu at (-127.5, -42.9)
- added H2: Mechanical_MountingHole, MountingHole:MountingHole_2.7mm_M2.5_ISO7380_Pad, F.Cu at (-127.5, 47.5)
- added H3: Mechanical_MountingHole, MountingHole:MountingHole_2.7mm_M2.5_ISO7380_Pad, F.Cu at (-71.0, 7.60)
- added H4: Mechanical_MountingHole, MountingHole:MountingHole_2.7mm_M2.5_ISO7380_Pad, F.Cu at (10.3, -64.1)
- added H5: Mechanical_MountingHole, MountingHole:MountingHole_2.7mm_M2.5_ISO7380_Pad, F.Cu at (0.00, 29.8)
- added H6: Mechanical_MountingHole, MountingHole:MountingHole_2.7mm_M2.5_ISO7380_Pad, F.Cu at (71.0, 7.60)
- added H7: Mechanical_MountingHole, MountingHole:MountingHole_2.7mm_M2.5_ISO7380_Pad, F.Cu at (155.0, 0.00)
- added H8: Mechanical_MountingHole, MountingHole:MountingHole_2.7mm_M2.5_ISO7380_Pad, F.Cu at (234.5, -48.4)
- added H9: Mechanical_MountingHole, MountingHole:MountingHole_2.7mm_M2.5_ISO7380_Pad, F.Cu at (234.5, 47.5)
- added RLEDL4: 1M, citrouille90 footprints:R_805, B.Cu at (-9.30, -64.8)
- C9: value 4,7u -> 4.7u
Routing:
- net Net-(J3-Shield): track 0.00 -> 18.6 mm
- net COL4: track 431.9 -> 434.2 mm
- net COL2: track 347.2 -> 349.3 mm
- net encB: track 155.0 -> 156.8 mm
- net COL9: track 662.7 -> 664.4 mm
- net led2: track 182.4 -> 180.7 mm
- net COL6: track 507.4 -> 509.0 mm
- net COL8: track 610.6 -> 612.0 mm
- net encA: track 156.9 -> 155.5 mm
- net COL7: track 572.2 -> 573.4 mm
- net ROW8: track 279.7 -> 280.7 mm
- net COL5: track 470.9 -> 471.8 mm
- net ROW1: track 203.7 -> 204.3 mm
- net COL3: track 353.6 -> 353.1 mm
- net +5V: track 185.2 -> 184.7 mm
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Other:
- board text added: "5V"
- board text added: "GND"
- board text added: "UPDI"

Commit message: Fine tune PCB
Parts:
- renumbered F2 to Fuse, ENC1 to PES12, RLEDL4 to R5, SWPB1 to RESET, J3 to USB, U2 to USBLC6
Other:
- board text added: "Rev A - 2026.03"
