File: kbpcb/pcb/Citrouille90/citrouille90.kicad_sch (KiCad schematic)
At the start: 19 parts, among them J1 3 pin connector, J3 USB mini b connector, U1 AVR64DU32-I/PT, U2 USBLC6-2SC6

Commit message: PCB work
Parts:
- removed J3: USB mini b connector, citrouille90 footprints:usb mini connector, symbol CitrouilleSymbolLibrary:USB mini b connector
- added C3: 4.7n, capacitors:C_0805_2012Metric_Pad1.18x1.45mm_HandSolder, symbol Device:C_Small
- added H1, H2, H3, H4, H5, H6, H7, H8, H9: Mechanical_MountingHole, MountingHole:MountingHole_2.7mm_M2.5_ISO7380_Pad, symbol CitrouilleSymbolLibrary:Mechanical_MountingHole
- added J3: USB mini b connector, citrouille90 footprints:usb mini connector, symbol Connector:USB_B_Mini
- added RLEDL4: 1M, citrouille90 footprints:R_805, symbol PCM_Resistor_AKL:R_0805
- C9: value 4,7u -> 4.7u
Connections:
- net D in+: now also J3.3 (D+)
- net D in-: now also J3.2 (D-)
- net GND: now also C3.1, J3.5 (GND), RLEDL4.2
- net VBUS: now also J3.1 (VBUS)
- new net: C3.2, J3.6 (Shield), RLEDL4.1
Other:
- moved on the sheet: C6, U2

Commit message: Fine tune PCB
Parts:
- renumbered RLEDL4 to R5
Changed lines of the file:
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@@
 		(on_board yes)
 		(dnp no)
-		(property "Reference" "RLEDL4"
+		(property "Reference" "R5"
 			(at 33.02 45.974 90)
 			(effects
@@
 			(project "citrouille90"
 				(path "/c86327b6-dcc1-4fd8-bf25-f8809a0ceda7"
-					(reference "RLEDL4")
+					(reference "R5")
 					(unit 1)
 				)
