File: kbpcb/pcb/Citrouille90/matrix.kicad_sch (KiCad schematic)
At the start: 181 parts

Commit message: Add RC filter to encoder
Parts:
- added C10, C11: 10n, capacitors:C_0805_2012Metric_Pad1.18x1.45mm_HandSolder, symbol Device:C_Small
- added R10, R11, R12, R13: 10K, citrouille90 footprints:R_805, symbol PCM_Resistor_AKL:R_0805
Connections:
- net GND: now also C10.2, C11.1
- net encA: now also C10.1, R10.1; no longer ENC1.A1
- net encB: now also C11.2, R11.1; no longer ENC1.B1
- new net: ENC1.A1, R10.2, R12.2
- new net: ENC1.B1, R11.2, R13.2
- new net +5V: R12.1, R13.1
Other:
- moved on the sheet: ENC1
